Commit message: Refactor tool management and update launch configurations for detachable tools

File: config/rbvogui_plus.ros2_control.xacro (robot description, xacro)
@@ -49,11 +49,4 @@
                 <state_interface name="velocity"/>
             </joint>
-            <joint name="robot_arm_rg6_finger_joint">
-                <command_interface name="position"/>
-                <state_interface name="position">
-                  <param name="initial_value">${initial_positions['robot_arm_rg6_finger_joint']}</param>
-                </state_interface>
-                <state_interface name="velocity"/>
-            </joint>
         </ros2_control>
     </xacro:macro>

File: config/rbvogui_plus.urdf.xacro (robot description, xacro)
@@ -2,7 +2,10 @@
 <robot xmlns:xacro="http://www.ros.org/wiki/xacro" name="rbvogui_plus">
     <xacro:arg name="initial_positions_file" default="initial_positions.yaml" />
-    <!-- Import rbvogui_plus urdf file -->
+    <!-- Detachable-tool scheme: bare arm, no baked end-effector -->
+    <xacro:arg name="end_effector"    default="none" />
+    <xacro:arg name="use_tool_changer" default="true" />
+    <!-- Import rbvogui_plus urdf file (end_effector and use_tool_changer flow via xacro args) -->
     <xacro:include filename="$(find robotnik_description)/robots/rbvogui/rbvogui_plus.urdf.xacro" />
-    <!-- Import control_xacro -->
+    <!-- FakeSystem ros2_control for MoveIt planning without Gazebo -->
     <xacro:include filename="rbvogui_plus.ros2_control.xacro" />
     <xacro:rbvogui_plus_ros2_control name="FakeSystem" initial_positions_file="$(arg initial_positions_file)"/>
